File: pcb/SumpPitNode/sumppitnodeboard.brd (EAGLE design)
At the start: 63.2 x 64.8 mm, 40 parts, among them IC1 7805T

Commit message: Save project.
Parts:
- removed LED_GREEN, LED_RED, LED_YELLOW: (no value), led:LED3MM
- added BIGLED_G, BIGLED_R, BIGLED_Y: (no value), SparkFun-Connectors:1X02
- added G_TR, R_TR, Y_TR: 2N3904, transistor:TO92
Connections:
- new net N$13: BIGLED_G.2, G_TR.3
- new net N$29: BIGLED_Y.2, Y_TR.3
- new net N$30: BIGLED_R.2, R_TR.3
- net GND: now also G_TR.1, R_TR.1, Y_TR.1; no longer LED_GREEN.K, LED_RED.K, LED_YELLOW.K
- net N$20: now also Y_TR.2; no longer LED_YELLOW.A
- net N$21: now also G_TR.2; no longer LED_GREEN.A
- net N$4: now also R_TR.2; no longer LED_RED.A
- net VCC_1: now also BIGLED_G.1, BIGLED_R.1, BIGLED_Y.1
Routing:
- net VCC_1: track 0.00 -> 184.0 mm, vias 0 -> 1
- net PIN_RPM_1: track 0.00 -> 110.1 mm
- net N$32: track 0.00 -> 91.0 mm
- net N$3: track 0.00 -> 86.7 mm, vias 0 -> 1
- net N$23: track 0.00 -> 74.3 mm, vias 0 -> 1
- net N$36: track 0.00 -> 65.3 mm, vias 0 -> 2
- net PIN_RPM_2: track 0.00 -> 56.8 mm, vias 0 -> 1
- net N$37: track 0.00 -> 56.7 mm, vias 0 -> 1
- net N$1: track 0.00 -> 51.0 mm
- net N$33: track 0.00 -> 48.5 mm
- net N$22: track 0.00 -> 45.1 mm, vias 0 -> 1
- net 3V3: track 0.00 -> 42.5 mm
- net PIN_VOLT_1: track 0.00 -> 41.3 mm
- net N$15: track 0.00 -> 38.9 mm, vias 0 -> 1
- net N$35: track 0.00 -> 37.2 mm
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